File: ClassicII.kicad_sch (KiCad schematic)
At the start: 72 parts, among them J11 POWER/ANALOG, J15 BURN-IN, J2 MODEM, J3 PRINTER

Commit message: More cleanup and cosmetic fixes
Parts:
- removed J2: MODEM, Connector_Imports:TE_5749268-1_MINI_DIN_8_RA_Shield, symbol MyConnector:Mini-DIN-8_MountingHole
- removed J3: PRINTER, Connector_Imports:TE_5749268-1_MINI_DIN_8_RA_Shield, symbol MyConnector:Mini-DIN-8_MountingHole
- removed RC1, RC2: CMD115S0002, MyPackage:SOIC-20W_7.5x12.8mm_P1.27mm_RC, symbol AppleASIC:RC_Network
- removed TP1: TestPoint, TestPoint:TestPoint_Pad_1.5x1.5mm, symbol Connector:TestPoint
- removed TP17, TP19, TP20, TP21, TP22, TP23, TP48, TP49, TP50, TP51, TP52, TP53, TP54, TP55, TP56, TP57: ~, TestPoint:TestPoint_THTPad_D1.0mm_Drill0.5mm, symbol Connector:TestPoint
- added C90: 680pF (W1), MyPackage:SMD_0603_1608Metric_Pad1.52x1.02mm, symbol Device:C_Small
- added C97: 680pF (W2), MyPackage:SMD_1206_3216Metric_Pad1.65x1.27mm, symbol Device:C_Small
- added L10: L_Ferrite_Small, MyPackage:L_2010_5025Metric_Pad2.0x2.2mm_HandSolder, symbol Device:L_Ferrite_Small
- added R49, R76: 47, MyPackage:SMD_0805_2012Metric_Pad1.25x1.65mm, symbol Device:R_Small_US
- added R85: 1200, MyPackage:SMD_0805_2012Metric_Pad1.25x1.65mm, symbol Device:R_Small_US
Connections:
- net Serial/RxDA- is gone; now on net RxDA-: J15.4 (Pin_4)
- net Serial/TxDA+ is gone; now on net TxDA+: J15.1 (Pin_1)
- net Serial/TxDA- is gone; now on net TxDA-: J15.2 (Pin_2)
- net GND: now also C90.1, C97.1, R85.2
- net EAGLE/31MHz renamed SYSCLOCKIN
- net EAGLE/BURN7 renamed BURN7
- net EAGLE/PBL: no longer names the net of J11.9 (Pin_9)
- net EAGLE/PBL: now also R49.2
- net EAGLE/VIDEO: no longer names the net of J11.6 (Pin_6)
- net EAGLE/VIDEO: now also C90.2, L10.2
- net EAGLE/~{HSYNC}: no longer names the net of J11.5 (Pin_5)
- net EAGLE/~{HSYNC}: now also C97.2, R76.2
- net EAGLE/~{VSYNC} renamed ~{VSYNC}
- net Serial/RxDA+ renamed RxDA+
- net Sound/SPEAKER renamed SPEAKER
- new net PBL: R49.1
- new net VIDEO: L10.1, R85.1
- new net ~{HSYNC}: R76.1
- no-connect marks 4 -> 3
Other:
- sheet ROM & FPU renamed System ROM
- added sheet Expansion Slot (romfpu.kicad_sch)
- added sheet RAM Expansion (simm.kicad_sch)
- added sheet RAM Transceivers (xcvr.kicad_sch)
- added sheet Test Points (test.kicad_sch)
- sheet EAGLE ports: added none; removed 31MHz, BURN7, PBL, VIDEO, ~{HSYNC}, ~{VSYNC}
- sheet Serial ports: added none; removed GPIA, GPIB, HSKIA, HSKIB, HSKOA, HSKOB, RxDA+, RxDA-, RxDB+, RxDB-, TxDA+, TxDA-, TxDB+, TxDB-
- sheet Sound ports: added none; removed SPEAKER
- moved on the sheet: C100, C101, C102, C103, C104, C105, C106, C107, C111, C112, C113, C114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
