File: cpu.kicad_sch (KiCad schematic)
At the start: 59 parts, among them U16 68030

Commit message: More cleanup and cosmetic fixes
Parts:
- removed R16, R53: 4700, MyPackage:SMD_0805_2012Metric_Pad1.25x1.65mm, symbol Device:R_Small_US
- removed TP10, TP11, TP12, TP13, TP29, TP31, TP34, TP40, TP6, TP7, TP8, TP9: ~, TestPoint:TestPoint_THTPad_D1.0mm_Drill0.5mm, symbol Connector:TestPoint
- removed TP30, TP32, TP41, TP42, TP44, TP45: ~, TestPoint:TestPoint_Pad_D1.0mm, symbol Connector:TestPoint
- TP2, TP24, TP25, TP26, TP27, TP28, TP3, TP35, TP36, TP4, TP46, TP47, TP5: footprint TestPoint:TestPoint_THTPad_D1.0mm_Drill0.5mm -> MyPackage:TestPoint_THTPad_D1.0mm_Drill0.5mm
- TP33, TP37, TP38, TP39, TP43: footprint TestPoint:TestPoint_Pad_D1.0mm -> MyPackage:TestPoint_Pad_D1.0mm
Connections:
- net PHI renamed C16M_MICRO
Other:
- moved on the sheet: C63, C64, C65, C73, C74, C75, C78, C87, C88, L11, R41, R43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
