File: dfac.kicad_sch (KiCad schematic)
At the start: 23 parts, among them U4 DFAC

Commit message: More cleanup and cosmetic fixes
Parts:
- added TP134, TP136, TP148, TP159, TP160, TP162, TP69: ~, MyPackage:TestPoint_Pad_D1.0mm, symbol Connector:TestPoint
- added TP155, TP156, TP157, TP158: ~, MyPackage:TestPoint_THTPad_D1.0mm_Drill0.5mm, symbol Connector:TestPoint
- R42, R46: value 19100, 1% -> 19100 1%
- U4: value DFAC -> DFAC_343S1033
Connections:
- net AMPOUT: now reaches C72.2, R42.1, R46.1
- net AMPOUT: now also TP69.1
- net NFIN: now reaches C61.2, R42.2, U4.7 (NFIn)
- net NFIN: now also TP159.1
- net LPFOUTF: now reaches C41.2, R22.2, R25.1, R30.2, R31.1
- net LPFOUTF: now also TP148.1
- net PWMOUT: now reaches R25.2, U4.23 (PWMOut)
- net PWMOUT: now also TP160.1
- net LPFIN: now reaches C54.1, R31.2, U4.24 (LPFIn)
- net LPFIN: now also TP158.1
- net VHIGH: now reaches C45.1, C46.1, U4.28 (VHigh)
- net VHIGH: now also TP162.1
- net VLOW: now reaches C45.2, U4.27 (VLow)
- net VLOW: now also TP157.1
- net IVO: now reaches C69.2, R40.1, R46.2, U4.5 (IVO)
- net IVO: now also TP134.1
- net SCFO: now reaches C15.2, U4.12 (SCFOut)
- net SCFO: now also TP156.1
- net BYPASS: now reaches C11.1, U4.2 (Bypass)
- net BYPASS: now also TP155.1
- net at C53.1, R32.1, R35.2: now also TP136.1
- net DFAC15 renamed SND
- net DFAC16 renamed SAMP_CLK
- net DFAC17 renamed SER_CLK
- net EGRET22 renamed CLATCH
- net EGRET5 renamed CONF_CLK
- net ~{RESETSW} renamed CDATA
Other:
- moved on the sheet: C11, C12, C15, C41, C45, C46, C54, C61, C69, C72, R22, R25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
