File: eagle.kicad_sch (KiCad schematic)
At the start: 47 parts, among them U18 EAGLE

Commit message: More cleanup and cosmetic fixes
Parts:
- removed C35: 100pF (AZ), MyPackage:SMD_0603_1608Metric_Pad1.52x1.02mm, symbol Device:C_Small
- removed C90: 680pF (W1), MyPackage:SMD_0603_1608Metric_Pad1.52x1.02mm, symbol Device:C_Small
- removed C97: 680pF (W2), MyPackage:SMD_1206_3216Metric_Pad1.65x1.27mm, symbol Device:C_Small
- removed L10: L_Ferrite_Small, MyPackage:L_2010_5025Metric_Pad2.0x2.2mm_HandSolder, symbol Device:L_Ferrite_Small
- removed R10, R11, R49, R76: 47, MyPackage:SMD_0805_2012Metric_Pad1.25x1.65mm, symbol Device:R_Small_US
- removed R52, R56, R58, R61, R62, R63, R67, R68, R73, R74, R75, R78, R79, R81, R82, R87, R92, R94: 22, MyPackage:SMD_0805_2012Metric_Pad1.25x1.65mm, symbol Device:R_Small_US
- removed R85: 1200, MyPackage:SMD_0805_2012Metric_Pad1.25x1.65mm, symbol Device:R_Small_US
- removed TP60: ~, TestPoint:TestPoint_THTPad_D1.0mm_Drill0.5mm, symbol Connector:TestPoint
- added R16, R53: 4700, MyPackage:SMD_0805_2012Metric_Pad1.25x1.65mm, symbol Device:R_Small_US
- added TP149: ~, MyPackage:TestPoint_THTPad_D1.0mm_Drill0.5mm, symbol Connector:TestPoint
- TP14, TP15: footprint TestPoint:TestPoint_THTPad_D1.0mm_Drill0.5mm -> MyPackage:TestPoint_THTPad_D1.0mm_Drill0.5mm
Connections:
- net +5V: now also R16.1, R53.1
- net PBL: now also U18.106 (BRIGHT_PWM)
- net RA0: now also U18.7 (RA0)
- net RA1: now also U18.8 (RA1)
- net RA10: now also U18.121 (RA10)
- net RA2: now also U18.13 (RA2)
- net RA3: now also U18.21 (RA3)
- net RA4: now also U18.44 (RA4)
- net RA5: now also U18.79 (RA5)
- net RA6: now also U18.84 (RA6)
- net RA7: now also U18.99 (RA7)
- net RA8: now also U18.108 (RA8)
- net RA9: now also U18.116 (RA9)
- net VIDEO: now also R83.2
- net ~{CAS0H}: now also U18.83 (~{CAS3})
- net ~{CAS0L}: now also U18.119 (~{CAS2})
- net ~{CAS1H}: now also U18.80 (~{CAS1})
- net ~{CAS1L}: now also U18.117 (~{CAS0})
- net ~{DSACK1}: now also R53.2
- net ~{HSYNC}: now also U18.107 (~{HSYNC})
- net ~{IPL2}: now also R16.2
- net ~{RAS0}: now also U18.40 (~{RAS0})
- net ~{RAS1}: now also U18.24 (~{RAS1})
- net FDDWR: now reaches U18.100 (FDDWR)
- net ~{RAMRW}: now reaches U18.12 (RAMR/~{W})
- net 31MHz renamed SYSCLOCKIN
- net DFAC15 renamed SND
- net DFAC16 renamed SAMP_CLK
- net DFAC17 renamed SER_CLK
- net EAGLE_VCC1 renamed CORE2_PWR
- net EAGLE_VCC2 renamed CORE1_PWR
- net CORE1_PWR: now also TP149.1
- net EGRET10 renamed VIA_FULL
- net EGRET11 renamed XCVR_SESSION
- net EGRET23 renamed FAST_RESET
- net EGRET7 renamed VIA_DATA
- net EGRET8 renamed VIA_CLK
- net EGRET9 renamed SYS_SESSION
- net HDSEL renamed ~{HEADSEL}
- net PCLK renamed C3_7M
- net PHI renamed C16M_MICRO
- net PHI2 renamed C16M_SWIM
- net SWIMWRDATA renamed FDDWRIN
- net ~{CE1} renamed ~{SCC_SEL}
- net ~{CE2} renamed ~{SCSI_SEL}
- net ~{CE3} renamed ~{IWM_SEL}
- net ~{RAMEN} renamed ~{EN245}
- net ~{RD} renamed ~{IOR}
- net ~{ROMEN} renamed ~{ROM}
- net ~{WREQ} renamed ~{SCCWREQ}
- net ~{WR} renamed ~{IOW}
Other:
- moved on the sheet: C84, C91, C93, C99, L5, L6, R50, R59, R66, R71, R72, R77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
