File: egret.kicad_sch (KiCad schematic)
At the start: 36 parts, among them J6 ADB, Q1 MMBT3904, U10 EGRET, U12 LS1126, Y1 S3238E

Commit message: More schematic cleanup
Parts:
- U10: symbol AppleASIC:EGRET -> AppleASIC:EGRET_341S0851
- U12: value LS1126 -> LS1126 (343S0120); symbol Connector_Generic:Conn_02x04_Counter_Clockwise -> AppleASIC:LS1126_343S0120
Connections:
- no-connect marks 2 -> 3
Other:
- moved on the sheet: BT1, C13, C18, C22, C29, C30, C42, C47, C49, C55, C66, C70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

Commit message: More cleanup and cosmetic fixes
Parts:
- added TP152: ~, MyPackage:TestPoint_Pad_D1.0mm, symbol Connector:TestPoint
- added TP68, TP98: ~, MyPackage:TestPoint_THTPad_D1.0mm_Drill0.5mm, symbol Connector:TestPoint
- TP58: footprint TestPoint:TestPoint_THTPad_D1.0mm_Drill0.5mm -> MyPackage:TestPoint_THTPad_D1.0mm_Drill0.5mm
- U10: value EGRET -> EGRET_341S0851
Connections:
- net PRAM_RESET: now reaches C47.1, R26.2, U10.2 (~{RESET})
- net PRAM_RESET: now also TP98.1
- net FB: now reaches R48.2, R55.1, TP58.1
- net OSCO: now reaches R39.2, U10.4 (OSCO)
- net OSCO: now also TP152.1
- net at R17.1, U10.21 (PA5): now also TP68.1
- net EGRET10 renamed VIA_FULL
- net EGRET11 renamed XCVR_SESSION
- net EGRET22 renamed CLATCH
- net EGRET23 renamed FAST_RESET
- net EGRET5 renamed CONF_CLK
- net EGRET7 renamed VIA_DATA
- net EGRET8 renamed VIA_CLK
- net EGRET9 renamed SYS_SESSION
- net EGRET_VCC renamed EGRET_PWR
- net ~{RESETSW} renamed CDATA
Other:
- moved on the sheet: BT1, C13, C18, C22, C29, C30, C42, C47, C55, C66, C70, J6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
