File: floppy.kicad_sch (KiCad schematic)
At the start: 16 parts, among them J5 EXT FLOPPY, J9 INT FLOPPY, U9 SWIM

Commit message: More cleanup and cosmetic fixes
Parts:
- added C35: 100pF (AZ), MyPackage:SMD_0603_1608Metric_Pad1.52x1.02mm, symbol Device:C_Small
- added R10, R11: 47, MyPackage:SMD_0805_2012Metric_Pad1.25x1.65mm, symbol Device:R_Small_US
- added TP72: ~, MyPackage:TestPoint_Pad_D1.0mm, symbol Connector:TestPoint
Connections:
- net GND: now also C35.2
- net DRVWR: no longer names the net of J9.18 (Pin_18), RC3.9
- net DRVWR: now also R10.2
- net HDSEL renamed ~{HEADSEL}
- net PHI2 renamed C16M_SWIM
- net SWIMWRDATA renamed FDDWRIN
- net ~{CE3} renamed ~{IWM_SEL}
- new net FDDWR: R11.1
- new net WRFIL: C35.1, R10.1, R11.2, TP72.1
Other:
- moved on the sheet: U9
