File: rom.kicad_sch (KiCad schematic)
At the start: 8 parts, among them J10 ROM/FPU EXPANSION SLOT, J13 PROM select, U22 27C322, U23 27C322

Commit message: More cleanup and cosmetic fixes
Parts:
- removed J10: ROM/FPU EXPANSION SLOT, MyPackage:MacClassicROMFPU_2x25_P2.54mm_Vertical, symbol Connector_Generic:Conn_02x25_Odd_Even
- added TP138, TP139, TP140, TP141: ~, MyPackage:TestPoint_THTPad_D1.0mm_Drill0.5mm, symbol Connector:TestPoint
Connections:
- net at J13.5 (Pin_5), R90.1, U22.42 (A19)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: now also TP139.1, TP141.1
- net at J13.6 (Pin_6), R91.1, U22.1 (A18)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: now also TP138.1, TP140.1
- net ~{ROMEN} renamed ~{ROM}
Other:
- moved on the sheet: J13, R88, R90, R91, R96, U22, U23
