File: scsi.kicad_sch (KiCad schematic)
At the start: 12 parts, among them J4 EXT SCSI, J8 INT SCSI, U8 Am85C80

Commit message: More cleanup and cosmetic fixes
Parts:
- TP18: footprint TestPoint:TestPoint_THTPad_D1.0mm_Drill0.5mm -> MyPackage:TestPoint_THTPad_D1.0mm_Drill0.5mm
- U8: Desc (none) -> SCC; Desc2 (none) -> SCSI
Connections:
- net S_PUP renamed SCCSOFT5
- net ~{CE2} renamed ~{SCSI_SEL}
- net ~{RD} renamed ~{IOR}
- net ~{WR} renamed ~{IOW}
Other:
- moved on the sheet: C68, C71, L4, U8A
