File: sound.kicad_sch (KiCad schematic)
At the start: 53 parts, among them J1 SND OUT, J7 SND IN, Q2 MMBTA14, U1 MC34119, U11 LM3080, U2 78L08

Commit message: More cleanup and cosmetic fixes
Parts:
- added TP135, TP147: ~, MyPackage:TestPoint_THTPad_D1.0mm_Drill0.5mm, symbol Connector:TestPoint
- added TP94: ~, MyPackage:TestPoint_Pad_D1.0mm, symbol Connector:TestPoint
- TP16, TP59: footprint TestPoint:TestPoint_THTPad_D1.0mm_Drill0.5mm -> MyPackage:TestPoint_THTPad_D1.0mm_Drill0.5mm
Connections:
- net F1: now reaches C8.1, U1.3 (FC1)
- net F1: now also TP94.1
- net SNDI: now reaches C39.1, R24.1, R29.1, U1.4 (Vin)
- net SNDI: now also TP147.1
- net at C6.1, R6.2: now also TP135.1
Other:
- moved on the sheet: C10, C16, C17, C6, C62, J7, LP3, R5, R6, R7
