File: ClassicIIRevB/egret.kicad_sch (KiCad schematic)
At the start: 39 parts, among them J6 ADB, Q1 MMBT3904, U10 EGRET_341S0851, U12 LS1126 (343S0120), Y1 S3238E

Commit message: improved footprints and silkscreens
Parts:
- BT1: footprint MyPackage:BatteryHolder_0.5xAA -> MyPackage:BatteryHolder_Keystone_108_1_2xAA; symbol Device:Battery -> Device:Battery_Cell
Changed lines of the file:
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@@
 	(title_block
 		(title "Macintosh Classic II Revision B")
-		(date "2025-05-31")
+		(date "2025-06-04")
 		(company "Apple Computer")
 		(comment 1 "drawn by Bradley Bell")
@@
 	(wire
 		(pts
+			(xy 35.56 53.34) (xy 35.56 50.8)
+		)
+		(stroke
+			(width 0)
+			(type default)
+		)
+	)
+	(wire
+		(pts
 			(xy 68.58 111.76) (xy 38.1 111.76)
 		)
@@
 	)
 	(symbol
-		(lib_id "Device:Battery")
-		(at 35.56 55.88 0)
+		(lib_id "Device:Battery_Cell")
+		(at 35.56 58.42 0)
 		(mirror y)
 		(unit 1)
@@
 		(on_board yes)
 		(dnp no)
-		(fields_autoplaced yes)
 		(property "Reference" "BT1"
-			(at 31.75 54.0384 0)
+			(at 27.94 55.118 0)
 			(effects
 				(font
 					(size 1.27 1.27)
 				)
-				(justify left)
+				(justify right)
 			)
 		)
 		(property "Value" "3V"
-			(at 31.75 56.5784 0)
+			(at 27.94 57.658 0)
 			(effects
 				(font
 					(size 1.27 1.27)
 				)
-				(justify left)
+				(justify right)
 			)
 		)
-		(property "Footprint" "MyPackage:BatteryHolder_0.5xAA"
-			(at 35.56 54.356 90)
+		(property "Footprint" "MyPackage:BatteryHolder_Keystone_108_1_2xAA"
+			(at 35.56 56.896 90)
 			(effects
 				(font
@@
 		)
 		(property "Datasheet" "~"
-			(at 35.56 54.356 90)
+			(at 35.56 56.896 90)
 			(effects
 				(font
@@
 			)
 		)
-		(property "Description" "Multiple-cell battery"
-			(at 35.56 55.88 0)
+		(property "Description" "Single-cell battery"
+			(at 35.56 58.42 0)
 			(effects
 				(font

Commit message: Switch to some "official" net names
Parts:
- Q1: value MMBT3904 -> 2N3904 (MMBT3904)
- Y1: value S3238E -> 32.768K (S3238E)
- renumbered TP58 to TP109, TP68 to TP41, TP98 to TP71, TP152 to TP97
Connections:
- net PA5: now reaches R17.1, TP41.1, U10.21 (PA5)
- net FAST_RESET renamed ~{TESTEN}
- net ~{RST} renamed ~{RESET}
Other:
- moved on the sheet: TP41
Changed lines of the file:
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@@
 	(wire
 		(pts
+			(xy 101.6 101.6) (xy 109.22 101.6)
+		)
+		(stroke
+			(width 0)
+			(type default)
+		)
+	)
+	(wire
+		(pts
 			(xy 241.3 101.6) (xy 157.48 101.6)
 		)
@@
 		)
 	)
+	(label "PA5"
+		(at 101.6 101.6 0)
+		(effects
+			(font
+				(size 1.27 1.27)
+			)
+			(justify left bottom)
+		)
+	)
 	(label "FB"
 		(at 38.1 111.76 0)
@@
 		)
 	)
-	(global_label "FAST_RESET"
+	(global_label "~{TESTEN}"
 		(shape input)
 		(at 241.3 104.14 0)
@@
 		)
 	)
-	(global_label "~{RST}"
+	(global_label "~{RESET}"
 		(shape output)
 		(at 241.3 73.66 0)
@@
 		)
 		(property "Intersheetrefs" "${INTERSHEET_REFS}"
-			(at 247.7323 73.66 0)
+			(at 250.0303 73.66 0)
 			(effects
 				(font
@@
 	(symbol
 		(lib_id "Connector:TestPoint")
-		(at 109.22 101.6 90)
+		(at 101.6 101.6 90)
 		(mirror x)
 		(unit 1)
@@
 		(dnp no)
 		(fields_autoplaced yes)
-		(property "Reference" "TP68"
-			(at 105.918 97.79 90)
+		(property "Reference" "TP41"
+			(at 98.298 97.79 90)
 			(effects
 				(font
@@
 		)
 		(property "Value" "~"
-			(at 105.918 99.06 90)
+			(at 98.298 99.06 90)
 			(effects
 				(font
@@
 		)
 		(property "Footprint" "MyPackage:TestPoint_THTPad_D1.0mm_Drill0.5mm"
-			(at 109.22 106.68 0)
+			(at 101.6 106.68 0)
 			(effects
 				(font
@@
 		)
 		(property "Datasheet" "~"
-			(at 109.22 106.68 0)
+			(at 101.6 106.68 0)
 			(effects
 				(font
@@
 		)
 		(property "Description" "test point"
-			(at 109.22 101.6 0)
+			(at 101.6 101.6 0)
 			(effects
 				(font
@@
 			(project "ClassicIIRevB"
 				(path "/08c23af6-72f1-4a8f-a60c-b986fe71300f/040ed762-f009-4b79-aae0-9178ab7234ec"
-					(reference "TP68")
+					(reference "TP41")
 					(unit 1)
 				)
@@
 		(dnp no)
 		(fields_autoplaced yes)
-		(property "Reference" "TP58"
+		(property "Reference" "TP109"
 			(at 34.798 107.95 90)
 			(effects
@@
 			(project "ClassicIIRevB"
 				(path "/08c23af6-72f1-4a8f-a60c-b986fe71300f/040ed762-f009-4b79-aae0-9178ab7234ec"
-					(reference "TP58")
+					(reference "TP109")
 					(unit 1)
 				)
@@
 			)
 		)
-		(property "Value" "S3238E"
+		(property "Value" "32.768K (S3238E)"
 			(at 68.58 87.63 0)
 			(effects
@@
 		(dnp no)
 		(fields_autoplaced yes)
-		(property "Reference" "TP152"
+		(property "Reference" "TP97"
 			(at 33.02 116.2049 90)
 			(effects
@@
 			(project "ClassicIIRevB"
 				(path "/08c23af6-72f1-4a8f-a60c-b986fe71300f/040ed762-f009-4b79-aae0-9178ab7234ec"
-					(reference "TP152")
+					(reference "TP97")
 					(unit 1)
 				)
@@
 		(dnp no)
 		(fields_autoplaced yes)
-		(property "Reference" "TP98"
+		(property "Reference" "TP71"
 			(at 34.798 67.31 90)
 			(effects
@@
 			(project "ClassicIIRevB"
 				(path "/08c23af6-72f1-4a8f-a60c-b986fe71300f/040ed762-f009-4b79-aae0-9178ab7234ec"
-					(reference "TP98")
+					(reference "TP71")
 					(unit 1)
 				)
@@
 			)
 		)
-		(property "Value" "MMBT3904"
+		(property "Value" "2N3904 (MMBT3904)"
 			(at 180.34 123.1899 0)
 			(effects

Commit message: update exports
Other:
- title: Macintosh Classic II Revision B -> Macintosh Classic II (Later Revision)
Changed lines of the file:
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@@
 	(paper "USLetter")
 	(title_block
-		(title "Macintosh Classic II Revision B")
-		(date "2025-06-04")
+		(title "Macintosh Classic II (Later Revision)")
+		(date "2025-06-16")
 		(company "Apple Computer")
 		(comment 1 "drawn by Bradley Bell")

Commit message: Corrections to SMDs, more improved footprints
The later revision board reproduction design is now complete.
Parts:
- C13: value 47/16 -> 47uF 16V
- C18, C22, C29, C30: value 560pF (U2) -> 560pF
- C42, C47, C49, C55: value .1 (A5) -> 100nF
- C66: value 10pF (A1) -> 10pF
- C70: value 33pF (N1) -> 33pF
- Q1: value 2N3904 (MMBT3904) -> 2N3904; PartNum (none) -> MMBT3904
- R17: value 220 -> 220R
- R18, R36, R38, R84, R9: value 4700 -> 4.7K
- R3: value 4700 -> 470R
- R4: value 22 -> 22R
- R48, R55: value 1M -> 10M
- R97: value 0 -> 0R
- TP109, TP41, TP71, TP97: now left out of the parts list
- U10: value EGRET_341S0851 -> EGRET; PartNum (none) -> 341S0851
- U12: value LS1126 (343S0120) -> LS1126; PartNum (none) -> 343S0120
- Y1: value 32.768K (S3238E) -> 32.768K; PartNum (none) -> S3238E
Other:
- moved on the sheet: R19
Changed lines of the file:
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@@
 	(title_block
 		(title "Macintosh Classic II (Later Revision)")
-		(date "2025-06-16")
+		(date "2025-06-21")
 		(company "Apple Computer")
 		(comment 1 "drawn by Bradley Bell")
@@
 	(wire
 		(pts
-			(xy 162.56 111.76) (xy 162.56 114.3)
+			(xy 165.1 111.76) (xy 165.1 114.3)
 		)
 		(stroke
@@
 	(wire
 		(pts
-			(xy 162.56 119.38) (xy 162.56 121.92)
+			(xy 165.1 119.38) (xy 165.1 121.92)
 		)
 		(stroke
@@
 	(wire
 		(pts
-			(xy 162.56 121.92) (xy 170.18 121.92)
+			(xy 165.1 121.92) (xy 170.18 121.92)
 		)
 		(stroke
@@
 	(wire
 		(pts
-			(xy 162.56 111.76) (xy 157.48 111.76)
+			(xy 165.1 111.76) (xy 157.48 111.76)
 		)
 		(stroke
@@
 		(unit 1)
 		(exclude_from_sim no)
-		(in_bom yes)
+		(in_bom no)
 		(on_board yes)
 		(dnp no)
@@
 		(dnp no)
 		(property "Reference" "C30"
-			(at 221.488 150.368 0)
+			(at 221.234 150.368 0)
 			(effects
 				(font
@@
 			)
 		)
-		(property "Value" "560pF (U2)"
-			(at 221.488 152.908 0)
+		(property "Value" "560pF"
+			(at 221.234 152.908 0)
 			(effects
 				(font
@@
 			)
 		)
-		(property "Value" ".1 (A5)"
+		(property "Value" "100nF"
 			(at 53.34 83.8262 0)
 			(effects
@@
 			)
 		)
-		(property "Value" ".1 (A5)"
+		(property "Value" "100nF"
 			(at 99.06 55.8862 0)
 			(effects
@@
 	(symbol
 		(lib_id "Device:R_Small_US")
-		(at 162.56 116.84 0)
+		(at 165.1 116.84 0)
 		(mirror y)
 		(unit 1)
@@
 		(fields_autoplaced yes)
 		(property "Reference" "R19"
-			(at 165.1 115.5699 0)
+			(at 167.64 115.5699 0)
 			(effects
 				(font
@@
 		)
 		(property "Value" "1K"
-			(at 165.1 118.1099 0)
+			(at 167.64 118.1099 0)
 			(effects
 				(font
@@
 		)
 		(property "Footprint" "MyPackage:SMD_0805_2012Metric_Pad1.25x1.65mm"
-			(at 162.56 116.84 0)
+			(at 165.1 116.84 0)
 			(effects
 				(font
@@
 		)
 		(property "Datasheet" "~"
-			(at 162.56 116.84 0)
+			(at 165.1 116.84 0)
 			(effects
 				(font
@@
 		)
 		(property "Description" "Resistor, small US symbol"
-			(at 162.56 116.84 0)
+			(at 165.1 116.84 0)
 			(effects
 				(font
@@
 		(unit 1)
 		(exclude_from_sim no)
-		(in_bom yes)
+		(in_bom no)
 		(on_board yes)
 		(dnp no)
@@
 			)
 		)
-		(property "Value" "22"
+		(property "Value" "22R"
 			(at 185.42 113.03 90)
 			(effects
@@
 			)
 		)
-		(property "Value" "EGRET_341S0851"
+		(property "Value" "EGRET"
 			(at 144.3833 120.65 0)
 			(effects
@@
 			)
 		)
+		(property "PartNum" "341S0851"
+			(at 144.3833 125.73 0)
+			(effects
+				(font
+					(size 1.27 1.27)
+				)
+				(justify left)
+			)
+		)
 		(pin "1"
 		)
@@
 			)
 		)
-		(property "Value" "4700"
+		(property "Value" "470R"
 			(at 157.48 138.4299 0)
 			(effects
@@
 			)
 		)
-		(property "Value" "33pF (N1)"
+		(property "Value" "33pF"
 			(at 78.74 105.4162 0)
 			(effects
@@
 			)
 		)
-		(property "Value" "4700"
+		(property "Value" "4.7K"
 			(at 198.12 101.5999 0)
 			(effects
@@
 		(dnp no)
 		(property "Reference" "C29"
-			(at 233.934 155.448 0)
+			(at 234.442 156.464 0)
 			(effects
 				(font
@@
 			)
 		)
-		(property "Value" "560pF (U2)"
-			(at 233.934 157.988 0)
+		(property "Value" "560pF"
+			(at 234.442 159.004 0)
 			(effects
 				(font
@@
 			)
 		)
-		(property "Value" "1M"
+		(property "Value" "10M"
 			(at 72.39 95.25 90)
 			(effects
@@
 			)
 		)
-		(property "Value" ".1 (A5)"
+		(property "Value" "100nF"
 			(at 111.76 64.7762 0)
 			(effects
@@
 			)
 		)
-		(property "Value" "0"
+		(property "Value" "0R"
 			(at 187.96 100.33 90)
 			(effects
@@
 		(fields_autoplaced yes)
 		(property "Reference" "U12"
-			(at 65.6433 40.64 0)
+			(at 65.6433 38.1 0)
 			(effects
 				(font
@@
 			)
 		)
-		(property "Value" "LS1126 (343S0120)"
-			(at 65.6433 43.18 0)
+		(property "Value" "LS1126"
+			(at 65.6433 40.64 0)
 			(effects
 				(font
@@
 		)
 		(property "Description" "Battery Monitor"
-			(at 65.6433 45.72 0)
+			(at 65.6433 43.18 0)
 			(effects
 				(font
@@
 			)
 		)
+		(property "PartNum" "343S0120"
+			(at 65.6433 45.72 0)
+			(effects
+				(font
+					(size 1.27 1.27)
+				)
+				(justify left)
+			)
+		)
 		(pin "1"
 		)
@@
 		(fields_autoplaced yes)
 		(property "Reference" "Y1"
-			(at 68.58 85.09 0)
+			(at 68.58 82.55 0)
 			(effects
 				(font
@@
 			)
 		)
-		(property "Value" "32.768K (S3238E)"
-			(at 68.58 87.63 0)
+		(property "Value" "32.768K"
+			(at 68.58 85.09 0)
 			(effects
 				(font
@@
 			)
 		)
+		(property "PartNum" "S3238E"
+			(at 68.58 87.63 0)
+			(effects
+				(font
+					(size 1.27 1.27)
+				)
+			)
+		)
 		(pin "1"
 		)
@@
 			)
 		)
-		(property "Value" "560pF (U2)"
+		(property "Value" "560pF"
 			(at 213.36 156.2162 0)
 			(effects
@@
 			)
 		)
-		(property "Value" "4700"
+		(property "Value" "4.7K"
 			(at 78.74 33.0199 0)
 			(effects
@@
 			)
 		)
-		(property "Value" "47/16"
+		(property "Value" "47uF 16V"
 			(at 88.9 55.4481 0)
 			(effects
@@
 			)
 		)
-		(property "Value" ".1 (A5)"
+		(property "Value" "100nF"
 			(at 149.86 60.9662 0)
 			(effects
@@
 		(unit 1)
 		(exclude_from_sim no)
-		(in_bom yes)
+		(in_bom no)
 		(on_board yes)
 		(dnp no)
@@
 			)
 		)
-		(property "Value" "10pF (A1)"
+		(property "Value" "10pF"
 			(at 58.42 105.4162 0)
 			(effects
@@
 			)
 		)
-		(property "Value" "1M"
+		(property "Value" "10M"
 			(at 64.77 95.25 90)
 			(effects
@@
 			)
 		)
-		(property "Value" "4700"
+		(property "Value" "4.7K"
 			(at 147.32 138.4299 0)
 			(effects
@@
 		(unit 1)
 		(exclude_from_sim no)
-		(in_bom yes)
+		(in_bom no)
 		(on_board yes)
 		(dnp no)
@@
 			)
 		)
-		(property "Value" "4700"
+		(property "Value" "4.7K"
 			(at 116.84 92.71 90)
 			(effects
@@
 		(on_board yes)
 		(dnp no)
-		(fields_autoplaced yes)
 		(property "Reference" "C22"
 			(at 243.84 153.6762 0)
@@
 			)
 		)
-		(property "Value" "560pF (U2)"
+		(property "Value" "560pF"
 			(at 243.84 156.2162 0)
 			(effects
@@
 		(on_board yes)
 		(dnp no)
+		(fields_autoplaced yes)
 		(property "Reference" "Q1"
-			(at 180.34 120.6499 0)
+			(at 180.34 119.3799 0)
 			(effects
 				(font
@@
 			)
 		)
-		(property "Value" "2N3904 (MMBT3904)"
-			(at 180.34 123.1899 0)
+		(property "Value" "2N3904"
+			(at 180.34 121.9199 0)
 			(effects
 				(font
@@
 			)
 		)
+		(property "PartNum" "MMBT3904"
+			(at 180.34 124.4599 0)
+			(effects
+				(font
+					(size 1.27 1.27)
+				)
+				(justify left)
+			)
+		)
 		(pin "1"
 		)
@@
 			)
 		)
-		(property "Value" "4700"
+		(property "Value" "4.7K"
 			(at 83.82 72.3899 0)
 			(effects
@@
 			)
 		)
-		(property "Value" "220"
+		(property "Value" "220R"
 			(at 106.68 107.9499 0)
 			(effects
@@
 				(font
 					(size 1.27 1.27)
+					(thickness 0.254)
+					(bold yes)
 				)
 			)
