File: ClassicIIRevB/ram.kicad_sch (KiCad schematic)
At the start: 19 parts, among them U13 41464, U14 41464, U17 41464, U19 41464

Commit message: improved footprints and silkscreens
Parts:
- U13, U14, U17, U19: footprint MyPackage:SOJ-20_7.62x17.145mm_P1.27mm -> MyPackage:SOJ-26-20_7.62x17.145mm_P1.27mm; symbol MyRam:441000 -> MyRam:DRAM_1Mx4_26SOJ20
Connections:
- net +5V: now also U13.13 (VCC), U14.13 (VCC), U17.13 (VCC), U19.13 (VCC); no longer U13.10 (VCC), U14.10 (VCC), U17.10 (VCC), U19.10 (VCC)
- net BD18: now also U13.24 (DQ3); no longer U13.18 (DQ3)
- net BD19: now also U13.25 (DQ4); no longer U13.19 (DQ4)
- net BD22: now also U14.24 (DQ3); no longer U14.18 (DQ3)
- net BD23: now also U14.25 (DQ4); no longer U14.19 (DQ4)
- net BD26: now also U17.24 (DQ3); no longer U17.18 (DQ3)
- net BD27: now also U17.25 (DQ4); no longer U17.19 (DQ4)
- net BD30: now also U19.24 (DQ3); no longer U19.18 (DQ3)
- net BD31: now also U19.25 (DQ4); no longer U19.19 (DQ4)
- net BRA0: now also U13.9 (A0), U14.9 (A0), U17.9 (A0), U19.9 (A0); no longer U13.6 (A0), U14.6 (A0), U17.6 (A0), U19.6 (A0)
- net BRA1: now also U13.10 (A1), U14.10 (A1), U17.10 (A1), U19.10 (A1); no longer U13.7 (A1), U14.7 (A1), U17.7 (A1), U19.7 (A1)
- net BRA2: now also U13.11 (A2), U14.11 (A2), U17.11 (A2), U19.11 (A2); no longer U13.8 (A2), U14.8 (A2), U17.8 (A2), U19.8 (A2)
- net BRA3: now also U13.12 (A3), U14.12 (A3), U17.12 (A3), U19.12 (A3); no longer U13.9 (A3), U14.9 (A3), U17.9 (A3), U19.9 (A3)
- net BRA4: now also U13.14 (A4), U14.14 (A4), U17.14 (A4), U19.14 (A4); no longer U13.11 (A4), U14.11 (A4), U17.11 (A4), U19.11 (A4)
- net BRA5: now also U13.15 (A5), U14.15 (A5), U17.15 (A5), U19.15 (A5); no longer U13.12 (A5), U14.12 (A5), U17.12 (A5), U19.12 (A5)
- net BRA6: now also U13.16 (A6), U14.16 (A6), U17.16 (A6), U19.16 (A6); no longer U13.13 (A6), U14.13 (A6), U17.13 (A6), U19.13 (A6)
- net BRA7: now also U13.17 (A7), U14.17 (A7), U17.17 (A7), U19.17 (A7); no longer U13.14 (A7), U14.14 (A7), U17.14 (A7), U19.14 (A7)
- net BRA8: now also U13.18 (A8), U14.18 (A8), U17.18 (A8), U19.18 (A8); no longer U13.15 (A8), U14.15 (A8), U17.15 (A8), U19.15 (A8)
- net GND: now also U13.22 (~{OE}), U13.26 (VSS), U14.22 (~{OE}), U14.26 (VSS), U17.22 (~{OE}), U17.26 (VSS), U19.22 (~{OE}), U19.26 (VSS); no longer U13.16 (~{OE}), U13.20 (VSS), U14.16 (~{OE}), U14.20 (VSS), U17.16 (~{OE}), U17.20 (VSS), U19.16 (~{OE}), U19.20 (VSS)
- new net: R52.2, U13.23 (~{CAS}), U14.23 (~{CAS})
- new net: R82.2, U17.23 (~{CAS}), U19.23 (~{CAS})
Changed lines of the file:
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@@
 	(title_block
 		(title "Macintosh Classic II Revision B")
-		(date "2025-05-31")
+		(date "2025-06-04")
 		(company "Apple Computer")
 		(comment 1 "drawn by Bradley Bell")
@@
 	)
 	(symbol
-		(lib_id "MyRam:441000")
+		(lib_id "MyRam:DRAM_1Mx4_26SOJ20")
 		(at 86.36 85.09 0)
 		(unit 1)
@@
 			)
 		)
-		(property "Footprint" "MyPackage:SOJ-20_7.62x17.145mm_P1.27mm"
+		(property "Footprint" "MyPackage:SOJ-26-20_7.62x17.145mm_P1.27mm"
 			(at 59.69 116.84 0)
 			(effects
@@
 			)
 		)
-		(pin "6"
+		(pin "24"
 		)
-		(pin "7"
+		(pin "25"
 		)
-		(pin "8"
+		(pin "23"
 		)
 		(pin "13"
@@
 		(pin "10"
 		)
-		(pin "20"
+		(pin "22"
 		)
 		(pin "1"
@@
 		(pin "18"
 		)
-		(pin "19"
+		(pin "26"
 		)
 		(pin "4"
@@
 	)
 	(symbol
-		(lib_id "MyRam:441000")
+		(lib_id "MyRam:DRAM_1Mx4_26SOJ20")
 		(at 215.9 85.09 0)
 		(unit 1)
@@
 			)
 		)
-		(property "Footprint" "MyPackage:SOJ-20_7.62x17.145mm_P1.27mm"
+		(property "Footprint" "MyPackage:SOJ-26-20_7.62x17.145mm_P1.27mm"
 			(at 189.23 116.84 0)
 			(effects
@@
 			)
 		)
-		(pin "6"
+		(pin "23"
 		)
-		(pin "7"
+		(pin "26"
 		)
-		(pin "8"
+		(pin "24"
 		)
 		(pin "13"
@@
 		(pin "10"
 		)
-		(pin "20"
+		(pin "25"
 		)
 		(pin "1"
@@
 		(pin "18"
 		)
-		(pin "19"
+		(pin "22"
 		)
 		(pin "4"
@@
 	)
 	(symbol
-		(lib_id "MyRam:441000")
+		(lib_id "MyRam:DRAM_1Mx4_26SOJ20")
 		(at 129.54 85.09 0)
 		(unit 1)
@@
 			)
 		)
-		(property "Footprint" "MyPackage:SOJ-20_7.62x17.145mm_P1.27mm"
+		(property "Footprint" "MyPackage:SOJ-26-20_7.62x17.145mm_P1.27mm"
 			(at 102.87 116.84 0)
 			(effects
@@
 			)
 		)
-		(pin "6"
+		(pin "23"
 		)
-		(pin "7"
+		(pin "22"
 		)
-		(pin "8"
+		(pin "26"
 		)
 		(pin "13"
@@
 		(pin "10"
 		)
-		(pin "20"
+		(pin "24"
 		)
 		(pin "1"
@@
 		(pin "18"
 		)
-		(pin "19"
+		(pin "25"
 		)
 		(pin "4"
@@
 	)
 	(symbol
-		(lib_id "MyRam:441000")
+		(lib_id "MyRam:DRAM_1Mx4_26SOJ20")
 		(at 172.72 85.09 0)
 		(unit 1)
@@
 			)
 		)
-		(property "Footprint" "MyPackage:SOJ-20_7.62x17.145mm_P1.27mm"
+		(property "Footprint" "MyPackage:SOJ-26-20_7.62x17.145mm_P1.27mm"
 			(at 146.05 116.84 0)
 			(effects
@@
 			)
 		)
-		(pin "6"
+		(pin "23"
 		)
-		(pin "7"
+		(pin "22"
 		)
-		(pin "8"
+		(pin "26"
 		)
 		(pin "13"
@@
 		(pin "10"
 		)
-		(pin "20"
+		(pin "24"
 		)
 		(pin "1"
@@
 		(pin "18"
 		)
-		(pin "19"
+		(pin "25"
 		)
 		(pin "4"

Commit message: Switch to some "official" net names
Connections:
- net BD16 renamed RD0
- net BD17 renamed RD1
- net BD18 renamed RD2
- net BD19 renamed RD3
- net BD20 renamed RD4
- net BD21 renamed RD5
- net BD22 renamed RD6
- net BD23 renamed RD7
- net BD24 renamed RD8
- net BD25 renamed RD9
- net BD26 renamed RD10
- net BD27 renamed RD11
- net BD28 renamed RD12
- net BD29 renamed RD13
- net BD30 renamed RD14
- net BD31 renamed RD15
- net ~{CAS0H} renamed ~{CAS1H}
- net ~{CAS0L} renamed ~{CAS1L}
- net ~{RAS0} renamed ~{RAS1}
Changed lines of the file:
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@@
+		)
+	)
+	(label "RD2"
+		(at 104.14 69.85 180)
+		(effects
+			(font
+				(size 1.27 1.27)
+			)
+			(justify right bottom)
 		)
 	)
@@
 		)
 	)
+	(label "RD0"
+		(at 104.14 64.77 180)
+		(effects
+			(font
+				(size 1.27 1.27)
+			)
+			(justify right bottom)
+		)
+	)
 	(label "BRA7"
 		(at 68.58 82.55 0)
@@
 		)
 	)
-	(label "BD16"
-		(at 104.14 64.77 180)
-		(effects
-			(font
-				(size 1.27 1.27)
-			)
-			(justify right bottom)
-		)
-	)
 	(label "RA2"
 		(at 43.18 66.04 0)
@@
 		)
 	)
-	(label "BD30"
-		(at 233.68 69.85 180)
-		(effects
-			(font
-				(size 1.27 1.27)
-			)
-			(justify right bottom)
-		)
-	)
 	(label "RA6"
 		(at 43.18 86.36 0)
@@
 		)
 	)
+	(label "RD7"
+		(at 147.32 72.39 180)
+		(effects
+			(font
+				(size 1.27 1.27)
+			)
+			(justify right bottom)
+		)
+	)
 	(label "BRA1"
 		(at 68.58 67.31 0)
@@
 		)
 	)
+	(label "RD13"
+		(at 233.68 67.31 180)
+		(effects
+			(font
+				(size 1.27 1.27)
+			)
+			(justify right bottom)
+		)
+	)
+	(label "RD6"
+		(at 147.32 69.85 180)
+		(effects
+			(font
+				(size 1.27 1.27)
+			)
+			(justify right bottom)
+		)
+	)
 	(label "BRA3"
 		(at 68.58 72.39 0)
@@
 		)
 	)
+	(label "RD9"
+		(at 190.5 67.31 180)
+		(effects
+			(font
+				(size 1.27 1.27)
+			)
+			(justify right bottom)
+		)
+	)
 	(label "BRA6"
 		(at 68.58 80.01 0)
@@
 		)
 	)
+	(label "RD12"
+		(at 233.68 64.77 180)
+		(effects
+			(font
+				(size 1.27 1.27)
+			)
+			(justify right bottom)
+		)
+	)
+	(label "RD14"
+		(at 233.68 69.85 180)
+		(effects
+			(font
+				(size 1.27 1.27)
+			)
+			(justify right bottom)
+		)
+	)
 	(label "BRA7"
 		(at 198.12 82.55 0)
@@
 		)
 	)
-	(label "BD21"
-		(at 147.32 67.31 180)
-		(effects
-			(font
-				(size 1.27 1.27)
-			)
-			(justify right bottom)
-		)
-	)
 	(label "BRA10"
 		(at 60.96 106.68 180)
@@
 		)
 	)
-	(label "BD28"
-		(at 233.68 64.77 180)
+	(label "RD11"
+		(at 190.5 72.39 180)
+		(effects
+			(font
+				(size 1.27 1.27)
+			)
+			(justify right bottom)
+		)
+	)
+	(label "RD1"
+		(at 104.14 67.31 180)
 		(effects
 			(font
@@
 		)
 	)
-	(label "BD27"
-		(at 190.5 72.39 180)
-		(effects
-			(font
-				(size 1.27 1.27)
-			)
-			(justify right bottom)
-		)
-	)
 	(label "RA7"
 		(at 43.18 91.44 0)
@@
 		)
 	)
+	(label "RD4"
+		(at 147.32 64.77 180)
+		(effects
+			(font
+				(size 1.27 1.27)
+			)
+			(justify right bottom)
+		)
+	)
+	(label "RD15"
+		(at 233.68 72.39 180)
+		(effects
+			(font
+				(size 1.27 1.27)
+			)
+			(justify right bottom)
+		)
+	)
 	(label "BRA1"
 		(at 111.76 67.31 0)
@@
 		)
 	)
-	(label "BD18"
-		(at 104.14 69.85 180)
-		(effects
-			(font
-				(size 1.27 1.27)
-			)
-			(justify right bottom)
-		)
-	)
 	(label "BRA0"
 		(at 68.58 64.77 0)
@@
 		)
 	)
-	(label "BD20"
-		(at 147.32 64.77 180)
-		(effects
-			(font
-				(size 1.27 1.27)
-			)
-			(justify right bottom)
-		)
-	)
 	(label "RA3"
 		(at 43.18 71.12 0)
@@
 		)
 	)
+	(label "RD5"
+		(at 147.32 67.31 180)
+		(effects
+			(font
+				(size 1.27 1.27)
+			)
+			(justify right bottom)
+		)
+	)
 	(label "BRA5"
 		(at 60.96 81.28 180)
@@
 		)
 	)
+	(label "RD8"
+		(at 190.5 64.77 180)
+		(effects
+			(font
+				(size 1.27 1.27)
+			)
+			(justify right bottom)
+		)
+	)
 	(label "BRA9"
 		(at 68.58 87.63 0)
@@
 		)
 	)
-	(label "BD24"
-		(at 190.5 64.77 180)
-		(effects
-			(font
-				(size 1.27 1.27)
-			)
-			(justify right bottom)
-		)
-	)
 	(label "BRA3"
 		(at 60.96 71.12 180)
@@
 		)
 	)
-	(label "BD25"
-		(at 190.5 67.31 180)
-		(effects
-			(font
-				(size 1.27 1.27)
-			)
-			(justify right bottom)
-		)
-	)
-	(label "BD23"
-		(at 147.32 72.39 180)
-		(effects
-			(font
-				(size 1.27 1.27)
-			)
-			(justify right bottom)
-		)
-	)
-	(label "BD26"
-		(at 190.5 69.85 180)
-		(effects
-			(font
-				(size 1.27 1.27)
-			)
-			(justify right bottom)
-		)
-	)
 	(label "BRA4"
 		(at 154.94 74.93 0)
@@
 		)
 	)
-	(label "BD29"
-		(at 233.68 67.31 180)
-		(effects
-			(font
-				(size 1.27 1.27)
-			)
-			(justify right bottom)
-		)
-	)
 	(label "BRA4"
 		(at 68.58 74.93 0)
@@
 		)
 	)
+	(label "RD10"
+		(at 190.5 69.85 180)
+		(effects
+			(font
+				(size 1.27 1.27)
+			)
+			(justify right bottom)
+		)
+	)
 	(label "BRA5"
 		(at 68.58 77.47 0)
@@
 		)
 	)
-	(label "BD31"
-		(at 233.68 72.39 180)
-		(effects
-			(font
-				(size 1.27 1.27)
-			)
-			(justify right bottom)
-		)
-	)
 	(label "BRA8"
 		(at 154.94 85.09 0)
@@
 		)
 	)
-	(label "BD17"
-		(at 104.14 67.31 180)
+	(label "RD3"
+		(at 104.14 72.39 180)
 		(effects
 			(font
@@
 		)
 	)
-	(label "BD19"
-		(at 104.14 72.39 180)
-		(effects
-			(font
-				(size 1.27 1.27)
-			)
-			(justify right bottom)
-		)
-	)
 	(label "BRA4"
 		(at 60.96 76.2 180)
@@
 		)
 	)
-	(label "BD22"
-		(at 147.32 69.85 180)
-		(effects
-			(font
-				(size 1.27 1.27)
-			)
-			(justify right bottom)
-		)
-	)
 	(label "BRA0"
 		(at 111.76 64.77 0)
@@
 		)
 	)
-	(global_label "~{CAS0H}"
+	(global_label "~{CAS1H}"
 		(shape input)
 		(at 38.1 124.46 180)
@@
 		)
 	)
-	(global_label "~{RAS0}"
+	(global_label "~{RAS1}"
 		(shape input)
 		(at 38.1 114.3 180)
@@
 		)
 	)
-	(global_label "BD[16..31]"
+	(global_label "RD[0..15]"
 		(shape output)
 		(at 241.3 134.62 0)
@@
 		)
 	)
-	(global_label "BD[16..31]"
+	(global_label "RD[0..15]"
 		(shape input)
 		(at 38.1 134.62 180)
@@
 		)
 	)
-	(global_label "~{CAS0L}"
+	(global_label "~{CAS1L}"
 		(shape input)
 		(at 38.1 119.38 180)

Commit message: update exports
Other:
- title: Macintosh Classic II Revision B -> Macintosh Classic II (Later Revision)
Changed lines of the file:
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@@
 	(paper "USLetter")
 	(title_block
-		(title "Macintosh Classic II Revision B")
-		(date "2025-06-04")
+		(title "Macintosh Classic II (Later Revision)")
+		(date "2025-06-16")
 		(company "Apple Computer")
 		(comment 1 "drawn by Bradley Bell")

Commit message: Corrections to SMDs, more improved footprints
The later revision board reproduction design is now complete.
Parts:
- R52, R56, R61, R62, R63, R67, R68, R73, R74, R75, R78, R81, R82, R87, R94: value 22 -> 22R
- U13, U14, U17, U19: value 41464 -> 1Mx4; PartNum (none) -> MCM54000A
Changed lines of the file:
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@@
 	(title_block
 		(title "Macintosh Classic II (Later Revision)")
-		(date "2025-06-16")
+		(date "2025-06-21")
 		(company "Apple Computer")
 		(comment 1 "drawn by Bradley Bell")
@@
 		)
 		(property "Intersheetrefs" "${INTERSHEET_REFS}"
-			(at 254.5662 134.62 0)
+			(at 253.3567 134.62 0)
 			(effects
 				(font
@@
 		)
 		(property "Intersheetrefs" "${INTERSHEET_REFS}"
-			(at 24.8338 134.62 0)
+			(at 26.0433 134.62 0)
 			(effects
 				(font
@@
 		)
 		(property "Intersheetrefs" "${INTERSHEET_REFS}"
-			(at 253.1753 50.8 0)
+			(at 254.4453 50.8 0)
 			(effects
 				(font
@@
 			)
 		)
-		(property "Value" "22"
+		(property "Value" "22R"
 			(at 45.72 110.49 90)
 			(effects
@@
 			)
 		)
-		(property "Value" "22"
+		(property "Value" "22R"
 			(at 53.34 115.57 90)
 			(effects
@@
 		(fields_autoplaced yes)
 		(property "Reference" "U13"
-			(at 88.5033 57.15 0)
+			(at 88.5033 52.07 0)
 			(effects
 				(font
@@
 			)
 		)
-		(property "Value" "41464"
-			(at 88.5033 59.69 0)
+		(property "Value" "1Mx4"
+			(at 88.5033 54.61 0)
 			(effects
 				(font
@@
 			)
 		)
-		(property "Description" "256k x 4 bit Dynamic RAM"
-			(at 86.36 72.39 0)
+		(property "Description" "RAM LL"
+			(at 88.5033 57.15 0)
 			(effects
 				(font
 					(size 1.27 1.27)
+					(thickness 0.254)
+					(bold yes)
 				)
-				(hide yes)
+				(justify left)
+			)
+		)
+		(property "PartNum" "MCM54000A"
+			(at 88.5033 59.69 0)
+			(effects
+				(font
+					(size 1.27 1.27)
+				)
+				(justify left)
 			)
 		)
@@
 		(fields_autoplaced yes)
 		(property "Reference" "U19"
-			(at 218.0433 57.15 0)
+			(at 218.0433 52.07 0)
 			(effects
 				(font
@@
 			)
 		)
-		(property "Value" "41464"
-			(at 218.0433 59.69 0)
+		(property "Value" "1Mx4"
+			(at 218.0433 54.61 0)
 			(effects
 				(font
@@
 			)
 		)
-		(property "Description" "256k x 4 bit Dynamic RAM"
-			(at 215.9 72.39 0)
+		(property "Description" "RAM HH"
+			(at 218.0433 57.15 0)
 			(effects
 				(font
 					(size 1.27 1.27)
+					(thickness 0.254)
+					(bold yes)
 				)
-				(hide yes)
+				(justify left)
+			)
+		)
+		(property "PartNum" "MCM54000A"
+			(at 218.0433 59.69 0)
+			(effects
+				(font
+					(size 1.27 1.27)
+				)
+				(justify left)
 			)
 		)
@@
 			)
 		)
-		(property "Value" "22"
+		(property "Value" "22R"
 			(at 49.53 53.848 90)
 			(effects
@@
 			)
 		)
-		(property "Value" "22"
+		(property "Value" "22R"
 			(at 49.53 84.328 90)
 			(effects
@@
 			)
 		)
-		(property "Value" "22"
+		(property "Value" "22R"
 			(at 45.72 125.73 90)
 			(effects
@@
 			)
 		)
-		(property "Value" "22"
+		(property "Value" "22R"
 			(at 49.53 74.168 90)
 			(effects
@@
 			)
 		)
-		(property "Value" "22"
+		(property "Value" "22R"
 			(at 53.34 58.928 90)
 			(effects
@@
 			)
 		)
-		(property "Value" "22"
+		(property "Value" "22R"
 			(at 53.34 89.408 90)
 			(effects
@@
 		(fields_autoplaced yes)
 		(property "Reference" "U14"
-			(at 131.6833 57.15 0)
+			(at 131.6833 52.07 0)
 			(effects
 				(font
@@
 			)
 		)
-		(property "Value" "41464"
-			(at 131.6833 59.69 0)
+		(property "Value" "1Mx4"
+			(at 131.6833 54.61 0)
 			(effects
 				(font
@@
 			)
 		)
-		(property "Description" "256k x 4 bit Dynamic RAM"
-			(at 129.54 72.39 0)
+		(property "Description" "RAM ML"
+			(at 131.6833 57.15 0)
 			(effects
 				(font
 					(size 1.27 1.27)
+					(thickness 0.254)
+					(bold yes)
 				)
-				(hide yes)
+				(justify left)
+			)
+		)
+		(property "PartNum" "MCM54000A"
+			(at 131.6833 59.69 0)
+			(effects
+				(font
+					(size 1.27 1.27)
+				)
+				(justify left)
 			)
 		)
@@
 		(fields_autoplaced yes)
 		(property "Reference" "U17"
-			(at 174.8633 57.15 0)
+			(at 174.8633 52.07 0)
 			(effects
 				(font
@@
 			)
 		)
-		(property "Value" "41464"
-			(at 174.8633 59.69 0)
+		(property "Value" "1Mx4"
+			(at 174.8633 54.61 0)
 			(effects
 				(font
@@
 			)
 		)
-		(property "Description" "256k x 4 bit Dynamic RAM"
-			(at 172.72 72.39 0)
+		(property "Description" "RAM MH"
+			(at 174.8633 57.15 0)
 			(effects
 				(font
 					(size 1.27 1.27)
+					(thickness 0.254)
+					(bold yes)
 				)
-				(hide yes)
+				(justify left)
+			)
+		)
+		(property "PartNum" "MCM54000A"
+			(at 174.8633 59.69 0)
+			(effects
+				(font
+					(size 1.27 1.27)
+				)
+				(justify left)
 			)
 		)
@@
 			)
 		)
-		(property "Value" "22"
+		(property "Value" "22R"
 			(at 60.96 120.65 90)
 			(effects
@@
 			)
 		)
-		(property "Value" "22"
+		(property "Value" "22R"
 			(at 49.53 64.008 90)
 			(effects
@@
 			)
 		)
-		(property "Value" "22"
+		(property "Value" "22R"
 			(at 53.34 79.248 90)
 			(effects
@@
 			)
 		)
-		(property "Value" "22"
+		(property "Value" "22R"
 			(at 53.34 69.088 90)
 			(effects
@@
 			)
 		)
-		(property "Value" "22"
+		(property "Value" "22R"
 			(at 53.34 99.568 90)
 			(effects
@@
 			)
 		)
-		(property "Value" "22"
+		(property "Value" "22R"
 			(at 49.53 104.648 90)
 			(effects
@@
 			)
 		)
-		(property "Value" "22"
+		(property "Value" "22R"
 			(at 49.53 94.488 90)
 			(effects
